File: KiCAD/Analogue Potential Divider.kicad_sch (KiCad schematic)
At the start: 8 parts

Commit message: .
Changed lines of the file:
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@@
-	(wire
-		(pts
-			(xy 146.05 53.34) (xy 135.89 53.34)
-		)
-		(stroke
-			(width 0)
-			(type default)
-		)
-	)
 	(wire
 		(pts
@@
 	(wire
 		(pts
+			(xy 135.89 73.66) (xy 146.05 73.66)
+		)
+		(stroke
+			(width 0)
+			(type default)
+		)
+	)
+	(wire
+		(pts
 			(xy 125.73 73.66) (xy 135.89 73.66)
 		)
@@
 	(wire
 		(pts
-			(xy 135.89 63.5) (xy 146.05 63.5)
-		)
-		(stroke
-			(width 0)
-			(type default)
-		)
-	)
-	(wire
-		(pts
 			(xy 125.73 76.2) (xy 125.73 73.66)
 		)
@@
 	(wire
 		(pts
-			(xy 146.05 73.66) (xy 135.89 73.66)
-		)
-		(stroke
-			(width 0)
-			(type default)
-		)
-	)
-	(wire
-		(pts
-			(xy 135.89 53.34) (xy 128.27 53.34)
+			(xy 128.27 53.34) (xy 146.05 53.34)
 		)
 		(stroke
@@
 	(wire
 		(pts
-			(xy 128.27 63.5) (xy 135.89 63.5)
+			(xy 128.27 63.5) (xy 146.05 63.5)
 		)
 		(stroke
@@
 		)
 	)
+	(netclass_flag ""
+		(length 1)
+		(shape round)
+		(at 140.97 63.5 0)
+		(fields_autoplaced yes)
+		(effects
+			(font
+				(size 1.524 1.524)
+			)
+			(justify left bottom)
+		)
+		(property "Net Class" "PCBway min 1 oz "
+			(at 141.5999 62.5 0)
+			(show_name no)
+			(do_not_autoplace no)
+			(effects
+				(font
+					(size 0.25 0.25)
+				)
+				(justify left)
+			)
+		)
+		(property "Component Class" ""
+			(at -10.16 -10.16 0)
+			(show_name no)
+			(do_not_autoplace no)
+			(effects
+				(font
+					(size 1.27 1.27)
+					(italic yes)
+				)
+			)
+		)
+	)
+	(netclass_flag ""
+		(length 1)
+		(shape round)
+		(at 140.97 53.34 0)
+		(fields_autoplaced yes)
+		(effects
+			(font
+				(size 1.524 1.524)
+			)
+			(justify left bottom)
+		)
+		(property "Net Class" "PCBway min 1 oz "
+			(at 141.5999 52.34 0)
+			(show_name no)
+			(do_not_autoplace no)
+			(effects
+				(font
+					(size 0.25 0.25)
+				)
+				(justify left)
+			)
+		)
+		(property "Component Class" ""
+			(at -10.16 -20.32 0)
+			(show_name no)
+			(do_not_autoplace no)
+			(effects
+				(font
+					(size 1.27 1.27)
+					(italic yes)
+				)
+			)
+		)
+	)
+	(netclass_flag ""
+		(length 1)
+		(shape round)
+		(at 140.97 73.66 0)
+		(fields_autoplaced yes)
+		(effects
+			(font
+				(size 1.524 1.524)
+			)
+			(justify left bottom)
+		)
+		(property "Net Class" "PCBway min 1 oz "
+			(at 141.5999 72.66 0)
+			(show_name no)
+			(do_not_autoplace no)
+			(effects
+				(font
+					(size 0.25 0.25)
+				)
+				(justify left)
+			)
+		)
+		(property "Component Class" ""
+			(at -10.16 0 0)
+			(show_name no)
+			(do_not_autoplace no)
+			(effects
+				(font
+					(size 1.27 1.27)
+					(italic yes)
+				)
+			)
+		)
+	)
