File: KiCAD/CIB - Mosaic Octopus.kicad_pcb (KiCad board)
At the start: 2 copper layers, 130.2 x 72.2 mm, 132 parts, among them J1 RH Bank, J2 Front Bank, J3 LH Bank, J4 DB25

Commit message: .
Parts:
- moved R1a28 183.2 mm to (153.7, 91.4), turned to 180 degrees
- moved JP54 182.5 mm to (150.5, 91.4)
- moved R1a32 174.8 mm to (153.7, 97.8), turned to 180 degrees
- moved JP62 174.5 mm to (150.5, 97.8)
- moved R1a20 174.1 mm to (153.7, 78.7), turned to 180 degrees
- moved JP38 173.9 mm to (150.5, 78.7)
- moved R1a27 173.2 mm to (146.7, 91.4), turned to 180 degrees
- moved R1b28 168.8 mm to (139.7, 91.4), turned to 180 degrees
- moved R1a31 165.4 mm to (146.7, 97.8), turned to 180 degrees
- moved R1a19 164.8 mm to (146.7, 78.7), turned to 180 degrees
- moved R1b27 160.9 mm to (134.6, 91.4), turned to 180 degrees
- moved R1b32 160.3 mm to (139.7, 97.8), turned to 180 degrees
- moved R1b20 159.6 mm to (139.7, 78.7), turned to 180 degrees
- moved R1a18 159.1 mm to (153.7, 75.6), turned to 180 degrees
- moved JP34 158.6 mm to (150.5, 75.6)
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Connections:
- J3 pad 1: /D4 -> /DIO4
- J3 pad 2: /D3 -> /DIO3
- J3 pad 3: /D2 -> /DIO2
- J3 pad 4: /D1 -> /DIO1
- J4 pad 13: unconnected-(J4-Pad13) -> /DIO4
- J4 pad 23: unconnected-(J4-P23-Pad23) -> /DIO1
- J4 pad 24: unconnected-(J4-P24-Pad24) -> /DIO2
- J4 pad 25: unconnected-(J4-P25-Pad25) -> /DIO3
Routing:
- net /A16: track 0.00 -> 97.4 mm
- net /ADC15: track 0.00 -> 95.9 mm
- net /ADC16: track 0.00 -> 94.8 mm
- net /A15: track 0.00 -> 91.8 mm
- net /A14: track 0.00 -> 90.3 mm
- net /ADC14: track 0.00 -> 86.9 mm
- net /ADC13: track 0.00 -> 86.6 mm
- net /A13: track 0.00 -> 83.5 mm
- net /A12: track 0.00 -> 82.1 mm
- net /ADC11: track 0.00 -> 79.2 mm
- net /ADC12: track 0.00 -> 78.3 mm
- net /A11: track 0.00 -> 75.6 mm
- net /A10: track 0.00 -> 74.2 mm
- net /ADC10: track 0.00 -> 69.7 mm
- net /ADC9: track 0.00 -> 69.4 mm
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Other:
- board size 130.2 x 72.2 mm -> 130.2 x 77.2 mm

Commit message: .
Parts:
- added U1: LM35-LP, Package_TO_SOT_THT:TO-92_Inline, F.Cu at (164.2, 68.2)
- turned JP5 to -90 degrees
- turned JP7 to -90 degrees
- turned JP8 to -90 degrees
Routing:
- net -5V: track 51.4 -> 200.0 mm
- net +5V: track 51.4 -> 199.7 mm, vias 16 -> 15
- net DG: track 0.00 -> 89.8 mm
- net /DIO1: track 0.00 -> 85.6 mm
- net +2V5: track 0.00 -> 84.5 mm
- net /DIO2: track 0.00 -> 77.6 mm
- net /DIO3: track 0.00 -> 67.4 mm
- net /DIO4: track 0.00 -> 57.4 mm
- net /ADC1: track 35.7 -> 71.1 mm
- net AG: track 51.4 -> 73.3 mm, vias 16 -> 15
- net /ADC15: track 95.9 -> 94.5 mm
- net /ADC11: track 79.2 -> 78.0 mm
- net /A3: track 53.5 -> 52.5 mm
- net /ADC5: track 52.7 -> 52.1 mm
- net Net-(JP5-B): track 14.2 -> 14.8 mm
- added copper zone on B.Cu, net AG
- added copper zone on F.Cu, net AG
