File: KiCAD/CIB - Mosaic Octopus.kicad_sch (KiCad schematic)
At the start: 4 parts, among them J1 RH Bank, J2 Front Bank, J3 LH Bank, J4 DB25

Commit message: .
Connections:
- net D1 is gone; now on net DIO1: J3.4 (Pin_4)
- net D2 is gone; now on net DIO2: J3.3 (Pin_3)
- net D3 is gone; now on net DIO3: J3.2 (Pin_2)
- net D4 is gone; now on net DIO4: J3.1 (Pin_1)
- net DIO4: now reaches J4.13
- net DIO1: now reaches J4.23 (P23)
- net DIO2: now reaches J4.24 (P24)
- net DIO3: now reaches J4.25 (P25)
Changed lines of the file:
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@@
+		)
+	)
+	(label "DIO1"
+		(at 40.64 146.05 0)
+		(effects
+			(font
+				(size 1.524 1.524)
+			)
+			(justify left bottom)
 		)
 	)
@@
 		)
 	)
-	(label "D2"
-		(at 40.64 148.59 0)
-		(effects
-			(font
-				(size 1.524 1.524)
-			)
-			(justify left bottom)
-		)
-	)
-	(label "D3"
-		(at 40.64 151.13 0)
-		(effects
-			(font
-				(size 1.524 1.524)
-			)
-			(justify left bottom)
-		)
-	)
 	(label "ADC10"
 		(at 250.19 43.18 180)
@@
 		)
 	)
+	(label "DIO4"
+		(at 40.64 153.67 0)
+		(effects
+			(font
+				(size 1.524 1.524)
+			)
+			(justify left bottom)
+		)
+	)
 	(label "A3"
 		(at 40.64 25.4 0)
@@
 		)
 	)
-	(label "D2"
-		(at 246.38 73.66 180)
+	(label "DIO3"
+		(at 40.64 151.13 0)
+		(effects
+			(font
+				(size 1.524 1.524)
+			)
+			(justify left bottom)
+		)
+	)
+	(label "DIO2"
+		(at 250.19 76.2 180)
 		(effects
 			(font
@@
 		)
 	)
-	(label "D3"
-		(at 246.38 76.2 180)
-		(effects
-			(font
-				(size 1.524 1.524)
-			)
-			(justify right bottom)
+	(label "DIO3"
+		(at 250.19 81.28 180)
+		(effects
+			(font
+				(size 1.524 1.524)
+			)
+			(justify right bottom)
+		)
+	)
+	(label "DIO2"
+		(at 40.64 148.59 0)
+		(effects
+			(font
+				(size 1.524 1.524)
+			)
+			(justify left bottom)
 		)
 	)
@@
 		)
 	)
-	(label "D1"
-		(at 246.38 71.12 180)
+	(label "DIO1"
+		(at 250.19 71.12 180)
 		(effects
 			(font
@@
 		)
 	)
-	(label "D4"
-		(at 40.64 153.67 0)
-		(effects
-			(font
-				(size 1.524 1.524)
-			)
-			(justify left bottom)
-		)
-	)
 	(label "ADC16"
 		(at 109.22 151.13 0)
@@
 		)
 	)
-	(label "D1"
-		(at 40.64 146.05 0)
-		(effects
-			(font
-				(size 1.524 1.524)
-			)
-			(justify left bottom)
-		)
-	)
 	(label "A7"
 		(at 73.66 71.12 180)
@@
 		)
 	)
-	(label "D4"
-		(at 246.38 78.74 180)
+	(label "DIO4"
+		(at 250.19 83.82 180)
 		(effects
 			(font
@@
 		)
 	)
+	(netclass_flag ""
+		(length 1)
+		(shape round)
+		(at 36.83 151.13 0)
+		(fields_autoplaced yes)
+		(effects
+			(font
+				(size 1.524 1.524)
+			)
+			(justify left bottom)
+		)
+		(property "Net Class" "PCBway min 1 oz "
+			(at 37.4599 150.13 0)
+			(show_name no)
+			(do_not_autoplace no)
+			(effects
+				(font
+					(size 0.25 0.25)
+				)
+				(justify left)
+			)
+		)
+		(property "Component Class" ""
+			(at -114.3 77.47 0)
+			(show_name no)
+			(do_not_autoplace no)
+			(effects
+				(font
+					(size 1.27 1.27)
+					(italic yes)
+				)
+			)
+		)
+	)
+	(netclass_flag ""
+		(length 1)
+		(shape round)
+		(at 36.83 146.05 0)
+		(fields_autoplaced yes)
+		(effects
+			(font
+				(size 1.524 1.524)
+			)
+			(justify left bottom)
+		)
+		(property "Net Class" "PCBway min 1 oz "
+			(at 37.4599 145.05 0)
+			(show_name no)
+			(do_not_autoplace no)
+			(effects
+				(font
+					(size 0.25 0.25)
+				)
+				(justify left)
+			)
+		)
+		(property "Component Class" ""
+			(at -114.3 72.39 0)
+			(show_name no)
+			(do_not_autoplace no)
+			(effects
+				(font
+					(size 1.27 1.27)
+					(italic yes)
+				)
+			)
+		)
+	)
+	(netclass_flag ""
+		(length 1)
+		(shape round)
+		(at 36.83 148.59 0)
+		(fields_autoplaced yes)
+		(effects
+			(font
+				(size 1.524 1.524)
+			)
+			(justify left bottom)
+		)
+		(property "Net Class" "PCBway min 1 oz "
+			(at 37.4599 147.59 0)
+			(show_name no)
+			(do_not_autoplace no)
+			(effects
+				(font
+					(size 0.25 0.25)
+				)
+				(justify left)
+			)
+		)
+		(property "Component Class" ""
+			(at -114.3 74.93 0)
+			(show_name no)
+			(do_not_autoplace no)
+			(effects
+				(font
+					(size 1.27 1.27)
+					(italic yes)
+				)
+			)
+		)
+	)
+	(netclass_flag ""
+		(length 1)
+		(shape round)
+		(at 36.83 153.67 0)
+		(fields_autoplaced yes)
+		(effects
+			(font
+				(size 1.524 1.524)
+			)
+			(justify left bottom)
+		)
+		(property "Net Class" "PCBway min 1 oz "
+			(at 37.4599 152.67 0)
+			(show_name no)
+			(do_not_autoplace no)
+			(effects
+				(font
+					(size 0.25 0.25)
+				)
+				(justify left)
+			)
+		)
+		(property "Component Class" ""
+			(at -114.3 80.01 0)
+			(show_name no)
+			(do_not_autoplace no)
+			(effects
+				(font
+					(size 1.27 1.27)
+					(italic yes)
+				)
+			)
+		)
+	)

Commit message: .
Parts:
- added U1: LM35-LP, Package_TO_SOT_THT:TO-92_Inline, symbol Sensor_Temperature:LM35-LP
Connections:
- net +5V: now also U1.1 (+V_{S})
- net ADC1: now also U1.2 (V_{OUT})
- net AG: now also U1.3 (GND)
