File: KiCAD/tmp/RTD Simulation - Pygmy Octopus/RTD Simulation.kicad_pcb (KiCad board)
At the start: 2 copper layers, 80.6 x 55.9 mm, 65 parts, among them J1 DA15, J2 Molex, J3 PT 3-4, J4 PT 1-2, J5 Enable, J6 Pin Header, J7 PT 1-2, Q1 PMV213SN, Q2 STN3NF06, Q3 STN3NF06, Q4 STN3NF06, Q5 STN3NF06, Q6 STN3NF06

Commit message: .
Parts:
- removed D11: SBR130S, Diode_SMD:D_SOD-323_HandSoldering
- removed D12: Red, LED_SMD:LED_0805_2012Metric_Pad1.15x1.40mm_HandSolder
- removed JP4: ~, Jumper:SolderJumper-3_P1.3mm_Bridged12_Pad1.0x1.5mm
- removed K6: ~, Relay_THT:Relay_DPDT_Omron_G6K-2P
- removed Q6: STN3NF06, Package_TO_SOT_SMD:SOT-23
- removed R22: ~, Resistor_SMD:R_1206_3216Metric_Pad1.30x1.75mm_HandSolder
- removed R23: 115R 0.1%, Resistor_SMD:R_1206_3216Metric_Pad1.30x1.75mm_HandSolder
- removed R24, R25: 1k, Resistor_SMD:R_0805_2012Metric_Pad1.20x1.40mm_HandSolder
- removed R26: 10k, Resistor_SMD:R_0805_2012Metric_Pad1.20x1.40mm_HandSolder
- JP1, JP2, JP3: footprint Jumper:SolderJumper-3_P1.3mm_Bridged12_Pad1.0x1.5mm -> Connector_PinHeader_2.54mm:PinHeader_1x03_P2.54mm_Vertical
- Q1: value PMV213SN -> STN3NF06; footprint Package_TO_SOT_SMD:SOT-23 -> Package_TO_SOT_SMD:SOT-223-3_TabPin2; moved to B.Cu
- Q2, Q3, Q4, Q5: footprint Package_TO_SOT_SMD:SOT-23 -> Package_TO_SOT_SMD:SOT-223-3_TabPin2; moved to B.Cu
- R1: value ~ -> 82.5R 0.1%
- R20: value 102R 0.1% -> ~
- moved R10 71.4 mm to (111.8, 57.8)
- moved R7 64.3 mm to (106.7, 57.8), turned to 180 degrees
- moved R6 63.6 mm to (111.8, 54.0)
- moved R8 63.5 mm to (106.7, 61.6), turned to 180 degrees
- moved R16 62.5 mm to (111.8, 65.4)
- moved D3 59.8 mm to (116.8, 55.9)
- moved R13 56.4 mm to (106.7, 65.4), turned to 180 degrees
- moved R14 55.6 mm to (106.7, 69.2), turned to 180 degrees
- moved R12 55.1 mm to (111.8, 61.6)
- moved R18 47.8 mm to (111.8, 69.2)
- moved R4 46.7 mm to (106.7, 54.0), turned to 180 degrees
- moved D6 42.7 mm to (111.8, 52.1), turned to 180 degrees
- moved R5 41.5 mm to (106.7, 52.1), turned to 0 degrees
- moved JP1 40.9 mm to (141.0, 40.6)
- moved D7 40.9 mm to (111.8, 55.9), turned to 180 degrees
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Connections:
- K4 pad 5: Net-(K4-Pad5) -> Net-(JP1-C)
- K5 pad 3: Net-(K4-Pad4) -> Net-(K4-Pad2)
- K5 pad 6: Net-(K4-Pad5) -> Net-(K4-Pad7)
- Q1 pad 2: GND -> /Relay_1
- Q1 pad 3: /Relay_1 -> GND
- Q2 pad 2: GND -> /Relay_2
- Q2 pad 3: /Relay_2 -> GND
- Q3 pad 2: GND -> /Relay_3
- Q3 pad 3: /Relay_3 -> GND
- Q4 pad 2: GND -> /Relay_4
- Q4 pad 3: /Relay_4 -> GND
- Q5 pad 2: GND -> /Relay_5
- Q5 pad 3: /Relay_5 -> GND
- R1 pad 2: Net-(K6-Pad4) -> Net-(K4-Pad4)
- R19 pad 1: Net-(JP2-B) -> Net-(JP2-A)
- R2 pad 1: Net-(JP2-A) -> Net-(JP2-B)
- R20 pad 2: Net-(K6-Pad4) -> Net-(K4-Pad4)
- R21 pad 1: Net-(JP3-B) -> Net-(JP3-A)
- R3 pad 1: Net-(JP3-A) -> Net-(JP3-B)
Routing:
- net +12V: track 6.91 -> 90.3 mm
- net /PT3 out: track 0.00 -> 73.6 mm
- net /PT1 out: track 0.00 -> 63.0 mm, vias 0 -> 1
- net /PT2 out: track 9.50 -> 66.9 mm, vias 0 -> 1
- net /PT4 out: track 8.53 -> 64.5 mm, vias 0 -> 2
- net /PT3 in: track 0.00 -> 55.8 mm, vias 0 -> 1
- net /PT1 in: track 0.00 -> 54.4 mm, vias 0 -> 1
- net /PT4 in: track 21.8 -> 68.1 mm
- net Net-(Q5-G): track 0.00 -> 36.3 mm, vias 0 -> 1
- net Net-(Q1-G): track 0.00 -> 35.1 mm, vias 0 -> 1
- net /Relay_4_en: track 0.00 -> 32.9 mm, vias 0 -> 2
- net /Relay_1_en: track 0.00 -> 32.8 mm
- net /Relay_3_en: track 0.00 -> 31.4 mm, vias 0 -> 1
- net /Relay_2_en: track 0.00 -> 31.4 mm
- net /PT2 in: track 21.7 -> 52.7 mm, vias 0 -> 1
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