File: KiCAD/tmp/RTD Simulation - Pygmy Octopus/RTD Simulation.kicad_sch (KiCad schematic)
At the start: 65 parts, among them J1 DA15, J2 Molex, J3 PT 3-4, J4 PT 1-2, J5 Enable, J6 Pin Header, J7 PT 1-2, Q1 PMV213SN, Q2 PMV213SN, Q3 PMV213SN, Q4 PMV213SN, Q5 PMV213SN, Q6 PMV213SN

Commit message: .
Parts:
- removed D11: SBR130S, Diode_SMD:D_SOD-323_HandSoldering, symbol Passive Components:Diode
- removed D12: Red, LED_SMD:LED_0805_2012Metric_Pad1.15x1.40mm_HandSolder, symbol Passive Components:LED
- removed JP1, JP4: ~, Jumper:SolderJumper-3_P1.3mm_Bridged12_Pad1.0x1.5mm, symbol Jumper:SolderJumper_3_Bridged12
- removed K6: ~, Relay_THT:Relay_DPDT_Omron_G6K-2P, symbol Relay:G2RL-2-DC24
- removed Q6: PMV213SN, Package_TO_SOT_SMD:SOT-23, symbol Device:Q_NMOS_GSD
- removed R22: ~, Resistor_SMD:R_1206_3216Metric_Pad1.30x1.75mm_HandSolder, symbol Passive Components:Resistor
- removed R23: 115R 0.1%, Resistor_SMD:R_1206_3216Metric_Pad1.30x1.75mm_HandSolder, symbol Passive Components:Resistor
- removed R24, R25: 1k, Resistor_SMD:R_0805_2012Metric_Pad1.20x1.40mm_HandSolder, symbol Passive Components:Resistor
- removed R26: 10k, Resistor_SMD:R_0805_2012Metric_Pad1.20x1.40mm_HandSolder, symbol Passive Components:Resistor
- added JP1: ~, Connector_PinHeader_2.54mm:PinHeader_1x03_P2.54mm_Vertical, symbol Jumper:Jumper_3_Open
- JP2, JP3: footprint Jumper:SolderJumper-3_P1.3mm_Bridged12_Pad1.0x1.5mm -> Connector_PinHeader_2.54mm:PinHeader_1x03_P2.54mm_Vertical; symbol Jumper:SolderJumper_3_Bridged12 -> Jumper:Jumper_3_Open
- Q1, Q2, Q3, Q4, Q5: value PMV213SN -> STN3NF06; footprint Package_TO_SOT_SMD:SOT-23 -> Package_TO_SOT_SMD:SOT-223-3_TabPin2; symbol Device:Q_NMOS_GSD -> Transistor_FET:NDT3055L
- R1: value ~ -> 82.5R 0.1%; DigiKey # P102BCCT-ND -> P82.5BCCT-ND; Farnell # 3269900 -> 3270121; Manufacturer # ERA-8AEB1020V -> ERA-8AEB82R5V; Mouser Part Number 667-ERA-8AEB1020V -> (none); now fitted
- R20: value 102R 0.1% -> ~; DigiKey # P102BCCT-ND -> P82.5BCCT-ND; Farnell # 3269900 -> 3270121; Manufacturer # ERA-8AEB1020V -> ERA-8AEB82R5V; Mouser Part Number 667-ERA-8AEB1020V -> (none); now not fitted
Connections:
- net GND: now also Q1.3 (S), Q2.3 (S), Q3.3 (S), Q4.3 (S), Q5.3 (S); no longer Q1.2 (S), Q2.2 (S), Q3.2 (S), Q4.2 (S), Q5.2 (S)
- net Relay_1: now also Q1.2 (D); no longer Q1.3 (D)
- net Relay_2: now also Q2.2 (D); no longer Q2.3 (D)
- net Relay_3: now also Q3.2 (D); no longer Q3.3 (D)
- net Relay_4: now also Q4.2 (D); no longer Q4.3 (D)
- net Relay_5: now also Q5.2 (D); no longer Q5.3 (D)
- net at JP2.1 (A): now also R19.1; no longer R2.1
- net at JP2.3 (B): now also R2.1; no longer R19.1
- net at K4.2: now also K5.3
- net at K4.4: now also R1.2, R20.2; no longer K5.3
- net at K4.5: now also JP1.2 (C); no longer K5.6
- net at K4.7: now also K5.6
- net at R21.1: now also JP3.1 (A); no longer JP3.3 (B)
- net at R20.1: now also JP1.1 (A)
- net at R1.1: now also JP1.3 (B)
- net at R3.1: now also JP3.3 (B); no longer JP3.1 (A)
- no-connect marks 1 -> 0
Other:
- note removed: "Jumpers to swap between PT100 and PT1000 values"
- moved on the sheet: D1, D10, D2, D3, D4, D5, D6, D7, D8, D9, K1, K2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
