File: KiCAD/tmp/Volt Free Contacts - Sandbird Octopus/Volt Free Contacts.kicad_pcb (KiCad board)
At the start: 2 copper layers, 159.6 x 100 mm, 62 parts, among them J1 DC37, J3 PT 3-4, J4 PT 1-2, J6 Pin Header, J7 03x32_DIN41612, Q1 STN3NF06, Q2 STN3NF06, Q3 STN3NF06, Q4 STN3NF06, Q5 STN3NF06

Commit message: .
Parts:
- removed D14, D15, D16, D17, D18, D19, D20, D21: SBR130S3-7, Diode_SMD:D_SOD-323_HandSoldering
- removed J7: 03x32_DIN41612, Eurocard:Eurocard
- removed K10, K11, K12, K13, K14, K15, K16, K9: ~, Relay_THT:Relay_DPDT_Omron_G6K-2P
- added H1: MountingHole, MountingHole:MountingHole_3.5mm_Pad, F.Cu at (95.2, 41.9)
- added H2: MountingHole, MountingHole:MountingHole_3.5mm_Pad, F.Cu at (158.8, 41.9)
- added H3: MountingHole, MountingHole:MountingHole_3.5mm_Pad, F.Cu at (95.2, 87.6)
- added H4: MountingHole, MountingHole:MountingHole_3.5mm_Pad, F.Cu at (158.8, 87.6)
- added J2: Molex, Connector_Molex:Molex_Micro-Fit_3.0_43045-1018_2x05-1MP_P3.00mm_Vertical, F.Cu at (135.9, 63.5)
- added J5: Enable, Connector_Molex:Molex_Micro-Fit_3.0_43045-1218_2x06-1MP_P3.00mm_Vertical, F.Cu at (97.8, 63.5)
- J1: value DC37 -> DA15; footprint Connector_Dsub:DSUB-37_Female_Horizontal_P2.77x2.84mm_EdgePinOffset9.90mm_Housed_MountingHolesOffset11.32mm -> Connector_Dsub:DSUB-9_Female_Horizontal_P2.77x2.84mm_EdgePinOffset7.70mm_Housed_MountingHolesOffset9.12mm
- J6, Q1, Q2, Q3, Q4, Q5: moved to B.Cu
- moved Q5 136.1 mm to (110.5, 48.3), turned to 180 degrees
- moved R9 124.6 mm to (106.7, 55.9)
- moved Q4 120.3 mm to (110.5, 55.9), turned to 180 degrees
- moved J3 120.2 mm to (132.1, 86.4)
- moved R6 117.5 mm to (111.8, 54.0)
- moved R15 117.3 mm to (106.7, 63.5)
- moved R7 116.8 mm to (106.7, 57.8), turned to 180 degrees
- moved R5 116.6 mm to (106.7, 52.1)
- moved J4 116.3 mm to (166.4, 108.0)
- moved R8 115.9 mm to (106.7, 61.6), turned to 180 degrees
- moved R4 111.7 mm to (106.7, 54.0), turned to 180 degrees
- moved J6 110.1 mm to (147.3, 58.4), turned to 180 degrees
- moved R12 110.0 mm to (111.8, 61.6)
- moved R13 109.5 mm to (106.7, 65.4), turned to 180 degrees
- moved R11 109.3 mm to (106.7, 59.7)
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Connections:
- J1 pad 0: unconnected-(J1-PAD-Pad0) -> GND
- J1 pad 1: /Ch1_com -> /PT1 in
- J1 pad 2: /Ch2_com -> /PT2 in
- J1 pad 3: unconnected-(J1-Pad3) -> /PT3 in
- J1 pad 4: unconnected-(J1-Pad4) -> /PT4 in
- J1 pad 5: unconnected-(J1-Pad5) -> /Pin_05
- J1 pad 6: unconnected-(J1-Pad6) -> /PT1 out
- J1 pad 7: unconnected-(J1-Pad7) -> /PT2 out
- J1 pad 8: unconnected-(J1-Pad8) -> /PT3 out
- J1 pad 9: unconnected-(J1-Pad9) -> /PT4 out
- K1 pad 5: /Ch1_no -> unconnected-(K1-Pad5)
- K1 pad 6: /Ch1_com -> unconnected-(K1-Pad6)
- K2 pad 5: /Ch2_no -> unconnected-(K2-Pad5)
- K2 pad 6: /Ch2_com -> unconnected-(K2-Pad6)
- K5 pad 2: unconnected-(K5-Pad2) -> /Relay_5
- K5 pad 4: unconnected-(K5-Pad4) -> /Relay_5
- K5 pad 5: unconnected-(K5-Pad5) -> /Relay_5
- K5 pad 7: unconnected-(K5-Pad7) -> /Relay_5
Routing:
- net /Ch2_com: track 162.1 -> 0.00 mm
- net /Ch2_no: track 161.5 -> 0.00 mm
- net /Ch1_no: track 153.9 -> 0.00 mm
- net /Ch1_com: track 152.2 -> 0.00 mm
- net +12V: track 0.00 -> 82.8 mm, vias 0 -> 1
- net /PT3 out: track 0.00 -> 52.7 mm
- net /PT4 out: track 0.00 -> 48.3 mm
- net /PT2 in: track 0.00 -> 46.6 mm, vias 0 -> 1
- net /PT3 in: track 0.00 -> 41.0 mm, vias 0 -> 1
- net /PT4 in: track 0.00 -> 38.8 mm
- net Net-(Q5-G): track 0.00 -> 36.3 mm, vias 0 -> 1
- net Net-(Q1-G): track 0.00 -> 35.1 mm, vias 0 -> 1
- net /PT1 out: track 0.00 -> 25.6 mm
- net /PT2 out: track 0.00 -> 25.5 mm
- net Net-(Q2-G): track 0.00 -> 22.9 mm, vias 0 -> 1
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- added copper zone on B.Cu, net GND
- added copper zone on F.Cu, net GND
Other:
- board size 159.6 x 100 mm -> 73 x 55.9 mm
