File: KiCAD/tmp/Volt Free Contacts - Sandbird Octopus/Volt Free Contacts.kicad_sch (KiCad schematic)
At the start: 62 parts, among them J1 DC37, J3 PT 3-4, J4 PT 1-2, J6 Pin Header, J7 03x32_DIN41612, Q1 STN3NF06, Q2 STN3NF06, Q3 STN3NF06, Q4 STN3NF06, Q5 STN3NF06

Commit message: .
Parts:
- removed D14, D15, D16, D17, D18, D19, D20, D21: SBR130S3-7, Diode_SMD:D_SOD-323_HandSoldering, symbol Device:D_Small_Filled
- removed J7: 03x32_DIN41612, Eurocard:Eurocard, symbol Eurocard:Conn_03x32_DIN41612
- removed K10, K11, K12, K13, K14, K15, K16, K9: ~, Relay_THT:Relay_DPDT_Omron_G6K-2P, symbol Relay:G2RL-2-DC24
- added H1, H2, H3, H4: MountingHole, MountingHole:MountingHole_3.5mm_Pad, symbol Mechanical:MountingHole_Pad
- added J2: Molex, Connector_Molex:Molex_Micro-Fit_3.0_43045-1018_2x05-1MP_P3.00mm_Vertical, symbol Connector_Generic:Conn_02x05_Top_Bottom
- added J5: Enable, Connector_Molex:Molex_Micro-Fit_3.0_43045-1218_2x06-1MP_P3.00mm_Vertical, symbol Connector_Generic:Conn_02x06_Top_Bottom
- J1: value DC37 -> DA15; footprint Connector_Dsub:DSUB-37_Female_Horizontal_P2.77x2.84mm_EdgePinOffset9.90mm_Housed_MountingHolesOffset11.32mm -> Connector_Dsub:DSUB-9_Female_Horizontal_P2.77x2.84mm_EdgePinOffset7.70mm_Housed_MountingHolesOffset9.12mm; symbol Connector:DC37_Receptacle_MountingHoles -> Connector:DE9_Receptacle_MountingHoles
Connections:
- net +12V: now also J5.7 (Pin_7)
- net GND: now also J1.0 (PAD), H1.1, H2.1, H3.1, H4.1, J2.10 (Pin_10), J5.12 (Pin_12), J5.6 (Pin_6)
- net PT1 in: now also J1.1, J2.1 (Pin_1)
- net PT1 out: now also J1.6, J2.6 (Pin_6)
- net PT2 in: now also J1.2, J2.2 (Pin_2)
- net PT2 out: now also J1.7, J2.7 (Pin_7)
- net PT3 in: now also J1.3, J2.3 (Pin_3)
- net PT3 out: now also J1.8, J2.8 (Pin_8)
- net PT4 in: now also J1.4, J2.4 (Pin_4)
- net PT4 out: now also J1.9, J2.9 (Pin_9)
- net Pin_05: now also J1.5, J2.5 (Pin_5)
- net Relay_1_en: now also J5.2 (Pin_2)
- net Relay_2_en: now also J5.3 (Pin_3)
- net Relay_3_en: now also J5.4 (Pin_4)
- net Relay_4_en: now also J5.5 (Pin_5)
- net Relay_5: now also K5.2, K5.4, K5.5, K5.7
- net Relay_5_en: now also J5.8 (Pin_8)
- net Ch1_com: no longer names the net of K1.6
- net Ch1_com: no longer J1.1
- net Ch1_no: no longer names the net of K1.5
- net Ch1_no: no longer J1.20
- net Ch2_com: no longer names the net of K2.6
- net Ch2_com: no longer J1.2
- net Ch2_no: no longer names the net of K2.5
- net Ch2_no: no longer J1.21
- new net +5V: J5.1 (Pin_1)
- new net Relay_6_en: J5.9 (Pin_9)
- new net Relay_7_en: J5.10 (Pin_10)
- new net Relay_8_en: J5.11 (Pin_11)
Other:
- note added: "Swap this out for a D25"
- note added: "https://chargepoint.atlassian.net/wiki/spaces/EN/pages/5094740380/Pygmy+Octopus"
- moved on the sheet: D1, D10, D11, D12, D13, D2, D3, D4, D5, D6, D7, D8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
